File: Hardware/WithGalvanicIsolation/SMC_FrontPanel_ExtensionBoard_Step2_V12_2.brd (EAGLE design)
At the start: 99.3 x 50.1 mm, 89 parts, among them J1 PIN2F061.060, J2 PIN2F061.060, J3 to mainboardconnector J3, J4 to Displaypanel, M1 ARDUINO-PRO-MINI-RAW, T1 BC857, T2 BC857, T3 BC857, T4 BC857, T5 BC857C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

Commit message: Fehlerbeseitigung siehe Readme
Parts:
- moved R28 0.16 mm to (75.4, 6.03), turned to 90 degrees
Connections:
- net DIRECTION_SW: now also M1.J6.11; no longer M1.J3.2
- net GND: now also M1.J3.1; no longer M1.J3.3
- net N$18: now also M1.J3.2; no longer M1.J3.1
Routing:
- net N$31: track 55.8 -> 33.4 mm, vias 2 -> 4
- net KEY: track 46.3 -> 29.7 mm, vias 1 -> 5
- net +5V: track 260.0 -> 246.6 mm, vias 17 -> 21
- net N$30: track 45.0 -> 32.9 mm, vias 3 -> 4
- net STOPLED_: track 34.2 -> 41.7 mm
- net DIRECTION_SW: track 40.7 -> 47.6 mm
- net N$17: track 26.1 -> 30.4 mm, vias 1 -> 2
- net N$18: track 44.5 -> 48.6 mm
- net DREHZAHL: track 11.5 -> 14.3 mm
- net N$4: track 15.2 -> 13.3 mm, vias 0 -> 1
- net N$15: track 19.9 -> 18.2 mm
- net SMC_SW: track 29.1 -> 30.7 mm
- net GND: track 317.6 -> 319.0 mm, vias 22 -> 20
- net ONEWIRE: track 37.8 -> 39.2 mm, vias 1 -> 5
- net STOPSW: track 32.6 -> 34.0 mm, vias 1 -> 2
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Other:
- board text added: "Revision V12.2"
- board text removed: "Revision V12.1"
