File: Hardware/WithGalvanicIsolation/SMC_FrontPanel_ExtensionBoard_Step2_V12_2.sch (EAGLE design)
At the start: 83 parts, among them J1 PIN2F061.060, J2 PIN2F061.060, J3 to mainboardconnector J3, J4 to Displaypanel, J9 JST-XH-02-PIN-ROUND-PAD, M1 ARDUINO-PRO-MINI-RAW, T1 BC857, T2 BC857, T3 BC857, T4 BC857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

Commit message: Fehlerbeseitigung siehe Readme
Connections:
- net DIRECTION_SW: now also M1.MOSI/PB3; no longer M1.ADC7
Other:
- note added: "12.2"
- note removed: "12.1"
Changed lines of the file:
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@@
 <setting verticaltext="up"/>
 </settings>
-<grid distance="0.05" unitdist="inch" unit="inch" style="lines" multiple="1" display="no" altdistance="0.01" altunitdist="inch" altunit="inch"/>
+<grid distance="0.1" unitdist="inch" unit="inch" style="lines" multiple="1" display="no" altdistance="0.01" altunitdist="inch" altunit="inch"/>
 <layers>
 <layer number="1" name="Top" color="4" fill="1" visible="no" active="no"/>
@@
 <text x="3.81" y="160.02" size="5.08" layer="97">Highvoltage Area</text>
 <text x="24.13" y="66.04" size="5.08" layer="97">Highvoltage Area</text>
-<text x="254" y="6.35" size="3.81" layer="97">12.1</text>
+<text x="254" y="6.35" size="3.81" layer="97">12.2</text>
 <text x="236.22" y="118.11" size="2.1844" layer="97">OLED Display</text>
 <text x="236.22" y="102.87" size="2.1844" layer="97">Rotary Encoder</text>
@@
 </instance>
 <instance part="P+5" gate="1" x="204.47" y="123.19" smashed="yes" rot="R90">
-<attribute name="VALUE" x="198.12" y="123.19" size="1.778" layer="96"/>
+<attribute name="VALUE" x="198.12" y="121.92" size="1.778" layer="96"/>
 </instance>
 <instance part="ENC" gate="-1" x="212.09" y="110.49" smashed="yes">
@@
 <net name="N$15" class="0">
 <segment>
-<pinref part="J2" gate="-1" pin="1"/>
-<wire x1="25.4" y1="15.24" x2="29.21" y2="15.24" width="0.1524" layer="91"/>
-<pinref part="F1" gate="G$1" pin="1"/>
-</segment>
-<segment>
 <pinref part="F2" gate="G$1" pin="1A"/>
 <wire x1="25.4" y1="-8.89" x2="21.59" y2="-8.89" width="0.1524" layer="91"/>
 <label x="21.59" y="-7.62" size="1.016" layer="95"/>
 </segment>
+<segment>
+<pinref part="J2" gate="-1" pin="1"/>
+<pinref part="F1" gate="G$1" pin="1"/>
+<wire x1="25.4" y1="15.24" x2="29.21" y2="15.24" width="0.1524" layer="91"/>
+</segment>
 </net>
 <net name="N$21" class="0">
-<segment>
-<pinref part="SV1" gate="G$1" pin="AC/N"/>
-<wire x1="39.37" y1="15.24" x2="105.41" y2="15.24" width="0.1524" layer="91"/>
-<pinref part="F1" gate="G$1" pin="2"/>
-</segment>
 <segment>
 <pinref part="F2" gate="G$1" pin="2A"/>
 <wire x1="35.56" y1="-8.89" x2="39.37" y2="-8.89" width="0.1524" layer="91"/>
 <label x="36.83" y="-7.62" size="1.016" layer="95"/>
+</segment>
+<segment>
+<pinref part="F1" gate="G$1" pin="2"/>
+<pinref part="SV1" gate="G$1" pin="AC/N"/>
+<wire x1="39.37" y1="15.24" x2="105.41" y2="15.24" width="0.1524" layer="91"/>
 </segment>
 </net>
@@
 <segment>
 <pinref part="R9" gate="G$1" pin="2"/>
-<label x="220.98" y="120.65" size="1.016" layer="95" xref="yes"/>
+<label x="226.06" y="120.65" size="1.016" layer="95" xref="yes"/>
 <wire x1="162.56" y1="123.19" x2="160.02" y2="123.19" width="0.1524" layer="91"/>
 <wire x1="160.02" y1="123.19" x2="160.02" y2="120.65" width="0.1524" layer="91"/>
@@
 </segment>
 <segment>
-<label x="220.98" y="118.11" size="1.016" layer="95" xref="yes"/>
+<label x="226.06" y="118.11" size="1.016" layer="95" xref="yes"/>
 <wire x1="157.48" y1="118.11" x2="209.55" y2="118.11" width="0.1524" layer="91"/>
 <pinref part="DISPLAY" gate="-4" pin="S"/>
@@
 <net name="DIRECTION_SW" class="0">
 <segment>
-<pinref part="M1" gate="G$1" pin="ADC7"/>
-<wire x1="86.36" y1="85.09" x2="93.98" y2="85.09" width="0.1524" layer="91"/>
-<label x="93.98" y="85.09" size="1.016" layer="95" xref="yes"/>
-</segment>
-<segment>
 <pinref part="R7" gate="G$1" pin="1"/>
 <pinref part="C1" gate="G$1" pin="2"/>
@@
 <junction x="186.69" y="163.83"/>
 <label x="181.61" y="163.83" size="1.016" layer="95" rot="R270" xref="yes"/>
+</segment>
+<segment>
+<pinref part="M1" gate="G$1" pin="MOSI/PB3"/>
+<wire x1="86.36" y1="92.71" x2="91.44" y2="92.71" width="0.1524" layer="91"/>
+<label x="92.71" y="92.71" size="1.016" layer="95" xref="yes"/>
 </segment>
 </net>
@@
 <text x="163.83" y="6.35" size="1.778" layer="97">Christian Brandtner , Paderborn, 05/2022
 Benutzung auf eigene Gefahr und Verantwortung</text>
-<text x="256.54" y="7.62" size="1.778" layer="97">12.1</text>
+<text x="256.54" y="7.62" size="1.778" layer="97">12.2</text>
 <text x="158.75" y="38.1" size="3.81" layer="97">Use at your own risk and responsibility</text>
 </plain>
